File: MCU DataLogger.kicad_pcb (KiCad board)
At the start: 2 copper layers, 51.2 x 30.9 mm, 29 parts, among them J1 Conn_01x04_Male, J2 Conn_01x04_Male, J3 Conn_01x09_Male, J4 Conn_02x03_Odd_Even, U1 24LC1025, U2 24LC1025, U3 DS1337S+, U4 ATMEGA328P-AU, Y1 32.768 KHz, Y2 16 MHz

Commit message: Fixed outstanding issues.
Parts:
- added REF**: KiCad-Logo2_5mm_SilkScreen, Symbol:KiCad-Logo2_5mm_SilkScreen, B.Cu at (64.0, 87.3)
Other:
- board text added: "VCC"

Commit message: Added gerber directories
Parts:
- renumbered REF** to REF1
Other:
- board text added: "0.2000 mm / 0.0000 mm"
- board text added: "0.3000 mm"
- board text added: "1.6000 mm"
- board text added: "51.2064 mm x 30.9372 mm"
- board text added: "BOARD CHARACTERISTICS"
- board text added: "Board Thickness:"
- board text added: "Board overall dimensions:"
- board text added: "Castellated pads:"
- board text added: "Copper Finish:"
- board text added: "Copper Layer Count:"
- board text added: "Edge card connectors:"
- board text added: "Impedance Control:"
- board text added: "Min hole diameter:"
- board text added: "Min track/spacing:"
- board text added: "No"
- board text added: "None"
- board text added: "Plated Board Edge:"
